File: hardware/atf1502as-plcc44-board/neogeo-diag-mvs-cha-atf1502as-plcc44.kicad_pcb (KiCad board)
At the start: 2 copper layers, 173.9 x 134 mm, 20 parts, among them J1 neogeo-mvs-cha-a-side-edge, J2 neogeo-mvs-cha-a-side-edge, J3 neogeo-mvs-cha-b-side-edge, J4 neogeo-mvs-cha-b-side-edge, J5 JTAG, U2 27C010 / 27C1001, U3 27C010 / 27C1001, U4 74HC574, U5 74HC574, U6 ATF1502AS-xJx44

Commit message: Some minor tweaks to schematics and pcbs
Other:
- board text added: "ATF150xAS"
- board text removed: "ATF1502AS"
Changed lines of the file:
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@@
     (descr "32-lead though-hole mounted DIP package, row spacing 15.24 mm (600 mils), Socket, LongPads")
     (tags "THT DIP DIL PDIP 2.54mm 15.24mm 600mil Socket LongPads")
-    (property "Sheetfile" "neogeo-diag-mvs-cha-plcc.kicad_sch")
+    (property "Sheetfile" "neogeo-diag-mvs-cha-atf1502as-plcc44.kicad_sch")
     (property "Sheetname" "")
     (property "ki_description" "27C010 1Mbit (128K x 8bit) EPROM")
@@
     (descr "SO, 20 Pin (https://www.ti.com/lit/ml/msop002a/msop002a.pdf), generated with kicad-footprint-generator ipc_gullwing_generator.py")
     (tags "SO SO")
-    (property "Sheetfile" "neogeo-diag-mvs-cha-plcc.kicad_sch")
+    (property "Sheetfile" "neogeo-diag-mvs-cha-atf1502as-plcc44.kicad_sch")
     (property "Sheetname" "")
     (property "ki_description" "OCTAL D FLIP-FLOP WITH CLEAR")
@@
     (descr "PLCC, 44 pins, through hole")
     (tags "plcc leaded")
-    (property "Sheetfile" "neogeo-diag-mvs-cha-plcc.kicad_sch")
+    (property "Sheetfile" "neogeo-diag-mvs-cha-atf1502as-plcc44.kicad_sch")
     (property "Sheetname" "")
     (property "ki_description" "Microchip CPLD, 32 Macrocell, 5 V, PLCC-44")
@@
     (descr "32-lead though-hole mounted DIP package, row spacing 15.24 mm (600 mils), Socket, LongPads")
     (tags "THT DIP DIL PDIP 2.54mm 15.24mm 600mil Socket LongPads")
-    (property "Sheetfile" "neogeo-diag-mvs-cha-plcc.kicad_sch")
+    (property "Sheetfile" "neogeo-diag-mvs-cha-atf1502as-plcc44.kicad_sch")
     (property "Sheetname" "")
     (property "ki_description" "27C010 1Mbit (128K x 8bit) EPROM")
@@
   (footprint "neogeo-diag:neogeo-mvs-a-side-edge" (layer "F.Cu")
     (at 156.100993 152.3)
-    (property "Sheetfile" "neogeo-diag-mvs-cha-plcc.kicad_sch")
+    (property "Sheetfile" "neogeo-diag-mvs-cha-atf1502as-plcc44.kicad_sch")
     (property "Sheetname" "")
     (property "ki_description" "NeoGeo MVS Prog A Side Gold Fingers Connector")
@@
     (descr "Through hole tests points for neogeo mvs prog board")
     (tags "Through hole tests points")
-    (property "Sheetfile" "neogeo-diag-mvs-cha-plcc.kicad_sch")
+    (property "Sheetfile" "neogeo-diag-mvs-cha-atf1502as-plcc44.kicad_sch")
     (property "Sheetname" "")
     (property "ki_description" "NeoGeo MVS Prog A Side Gold Fingers Connector")
@@
     (descr "Capacitor SMD 0805 (2012 Metric), square (rectangular) end terminal, IPC_7351 nominal, (Body size source: IPC-SM-782 page 76, https://www.pcb-3d.com/wordpress/wp-content/uploads/ipc-sm-782a_amendment_1_and_2.pdf, https://docs.google.com/spreadsheets/d/1BsfQQcO9C6DZCsRaXUlFlo91Tg2WpOkGARC1WS5S8t0/edit?usp=sharing), generated with kicad-footprint-generator")
     (tags "capacitor")
-    (property "Sheetfile" "neogeo-diag-mvs-cha-plcc.kicad_sch")
+    (property "Sheetfile" "neogeo-diag-mvs-cha-atf1502as-plcc44.kicad_sch")
     (property "Sheetname" "")
     (property "ki_description" "Capacitor symbol for simulation only")
@@
     (descr "Capacitor SMD 0805 (2012 Metric), square (rectangular) end terminal, IPC_7351 nominal, (Body size source: IPC-SM-782 page 76, https://www.pcb-3d.com/wordpress/wp-content/uploads/ipc-sm-782a_amendment_1_and_2.pdf, https://docs.google.com/spreadsheets/d/1BsfQQcO9C6DZCsRaXUlFlo91Tg2WpOkGARC1WS5S8t0/edit?usp=sharing), generated with kicad-footprint-generator")
     (tags "capacitor")
-    (property "Sheetfile" "neogeo-diag-mvs-cha-plcc.kicad_sch")
+    (property "Sheetfile" "neogeo-diag-mvs-cha-atf1502as-plcc44.kicad_sch")
     (property "Sheetname" "")
     (property "ki_description" "Capacitor symbol for simulation only")
@@
     (descr "SO, 20 Pin (https://www.ti.com/lit/ml/msop002a/msop002a.pdf), generated with kicad-footprint-generator ipc_gullwing_generator.py")
     (tags "SO SO")
-    (property "Sheetfile" "neogeo-diag-mvs-cha-plcc.kicad_sch")
+    (property "Sheetfile" "neogeo-diag-mvs-cha-atf1502as-plcc44.kicad_sch")
     (property "Sheetname" "")
     (property "ki_description" "OCTAL D FLIP-FLOP WITH CLEAR")
@@
     (descr "Capacitor SMD 0805 (2012 Metric), square (rectangular) end terminal, IPC_7351 nominal, (Body size source: IPC-SM-782 page 76, https://www.pcb-3d.com/wordpress/wp-content/uploads/ipc-sm-782a_amendment_1_and_2.pdf, https://docs.google.com/spreadsheets/d/1BsfQQcO9C6DZCsRaXUlFlo91Tg2WpOkGARC1WS5S8t0/edit?usp=sharing), generated with kicad-footprint-generator")
     (tags "capacitor")
-    (property "Sheetfile" "neogeo-diag-mvs-cha-plcc.kicad_sch")
+    (property "Sheetfile" "neogeo-diag-mvs-cha-atf1502as-plcc44.kicad_sch")
     (property "Sheetname" "")
     (property "ki_description" "Capacitor symbol for simulation only")
@@
     (descr "Capacitor SMD 0805 (2012 Metric), square (rectangular) end terminal, IPC_7351 nominal, (Body size source: IPC-SM-782 page 76, https://www.pcb-3d.com/wordpress/wp-content/uploads/ipc-sm-782a_amendment_1_and_2.pdf, https://docs.google.com/spreadsheets/d/1BsfQQcO9C6DZCsRaXUlFlo91Tg2WpOkGARC1WS5S8t0/edit?usp=sharing), generated with kicad-footprint-generator")
     (tags "capacitor")
-    (property "Sheetfile" "neogeo-diag-mvs-cha-plcc.kicad_sch")
+    (property "Sheetfile" "neogeo-diag-mvs-cha-atf1502as-plcc44.kicad_sch")
     (property "Sheetname" "")
     (property "ki_description" "Capacitor symbol for simulation only")
@@
     (descr "Capacitor SMD 0805 (2012 Metric), square (rectangular) end terminal, IPC_7351 nominal, (Body size source: IPC-SM-782 page 76, https://www.pcb-3d.com/wordpress/wp-content/uploads/ipc-sm-782a_amendment_1_and_2.pdf, https://docs.google.com/spreadsheets/d/1BsfQQcO9C6DZCsRaXUlFlo91Tg2WpOkGARC1WS5S8t0/edit?usp=sharing), generated with kicad-footprint-generator")
     (tags "capacitor")
-    (property "Sheetfile" "neogeo-diag-mvs-cha-plcc.kicad_sch")
+    (property "Sheetfile" "neogeo-diag-mvs-cha-atf1502as-plcc44.kicad_sch")
     (property "Sheetname" "")
     (property "ki_description" "Capacitor symbol for simulation only")
@@
     (descr "Through hole tests points for neogeo mvs prog board")
     (tags "Through hole tests points")
-    (property "Sheetfile" "neogeo-diag-mvs-cha-plcc.kicad_sch")
+    (property "Sheetfile" "neogeo-diag-mvs-cha-atf1502as-plcc44.kicad_sch")
     (property "Sheetname" "")
     (property "ki_description" "NeoGeo MVS Prog A Side Gold Fingers Connector")
@@
     (descr "Through hole straight pin header, 1x06, 2.54mm pitch, single row")
     (tags "Through hole pin header THT 1x06 2.54mm single row")
-    (property "Sheetfile" "neogeo-diag-mvs-cha-plcc.kicad_sch")
+    (property "Sheetfile" "neogeo-diag-mvs-cha-atf1502as-plcc44.kicad_sch")
     (property "Sheetname" "")
     (property "ki_description" "Generic connector, single row, 01x06, script generated")
@@
     (descr "Capacitor SMD 0805 (2012 Metric), square (rectangular) end terminal, IPC_7351 nominal, (Body size source: IPC-SM-782 page 76, https://www.pcb-3d.com/wordpress/wp-content/uploads/ipc-sm-782a_amendment_1_and_2.pdf, https://docs.google.com/spreadsheets/d/1BsfQQcO9C6DZCsRaXUlFlo91Tg2WpOkGARC1WS5S8t0/edit?usp=sharing), generated with kicad-footprint-generator")
     (tags "capacitor")
-    (property "Sheetfile" "neogeo-diag-mvs-cha-plcc.kicad_sch")
+    (property "Sheetfile" "neogeo-diag-mvs-cha-atf1502as-plcc44.kicad_sch")
     (property "Sheetname" "")
     (property "ki_description" "Capacitor symbol for simulation only")
@@
     (descr "Capacitor SMD 0805 (2012 Metric), square (rectangular) end terminal, IPC_7351 nominal, (Body size source: IPC-SM-782 page 76, https://www.pcb-3d.com/wordpress/wp-content/uploads/ipc-sm-782a_amendment_1_and_2.pdf, https://docs.google.com/spreadsheets/d/1BsfQQcO9C6DZCsRaXUlFlo91Tg2WpOkGARC1WS5S8t0/edit?usp=sharing), generated with kicad-footprint-generator")
     (tags "capacitor")
-    (property "Sheetfile" "neogeo-diag-mvs-cha-plcc.kicad_sch")
+    (property "Sheetfile" "neogeo-diag-mvs-cha-atf1502as-plcc44.kicad_sch")
     (property "Sheetname" "")
     (property "ki_description" "Capacitor symbol for simulation only")
@@
     (descr "Capacitor SMD 0805 (2012 Metric), square (rectangular) end terminal, IPC_7351 nominal, (Body size source: IPC-SM-782 page 76, https://www.pcb-3d.com/wordpress/wp-content/uploads/ipc-sm-782a_amendment_1_and_2.pdf, https://docs.google.com/spreadsheets/d/1BsfQQcO9C6DZCsRaXUlFlo91Tg2WpOkGARC1WS5S8t0/edit?usp=sharing), generated with kicad-footprint-generator")
     (tags "capacitor")
-    (property "Sheetfile" "neogeo-diag-mvs-cha-plcc.kicad_sch")
+    (property "Sheetfile" "neogeo-diag-mvs-cha-atf1502as-plcc44.kicad_sch")
     (property "Sheetname" "")
     (property "ki_description" "Capacitor symbol for simulation only")
@@
   (footprint "neogeo-diag:neogeo-mvs-b-side-edge" (layer "B.Cu")
     (at 153.560993 152.3 180)
-    (property "Sheetfile" "neogeo-diag-mvs-cha-plcc.kicad_sch")
+    (property "Sheetfile" "neogeo-diag-mvs-cha-atf1502as-plcc44.kicad_sch")
     (property "Sheetname" "")
     (property "ki_description" "NeoGeo MVS Prog A Side Gold Fingers Connector")
@@
     (effects (font (size 0.7 0.7) (thickness 0.12)) (justify left))
   )
-  (gr_text "ATF1502AS" (at 85.6234 80.4164) (layer "F.SilkS")
+  (gr_text "ATF150xAS" (at 85.6234 80.4164) (layer "F.SilkS")
     (effects (font (size 1 1) (thickness 0.15)) (justify left bottom))
   )
