File: hardware/atf1502as-plcc44-board/neogeo-diag-mvs-cha-atf1502as-plcc44.kicad_sch (KiCad schematic)
At the start: 18 parts, among them J1 neogeo-mvs-cha-a-side-edge, J2 neogeo-mvs-cha-a-side-edge, J3 neogeo-mvs-cha-b-side-edge, J4 neogeo-mvs-cha-b-side-edge, J5 JTAG, U2 27C010 / 27C1001, U3 27C010 / 27C1001, U4 74HC574, U5 74HC574, U6 ATF1502AS-xJx44

Commit message: Some minor tweaks to schematics and pcbs
Other:
- note added: "M1 ROM + Address Logic"
- note removed: "M1 ROM + CPLD (PLCC)"
Changed lines of the file:
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@@
     (effects (font (size 3 3)) (justify left bottom))
   )
-  (text "M1 ROM + CPLD (PLCC)" (at 290.83 147.955 0)
+  (text "M1 ROM + Address Logic" (at 284.48 146.05 0)
     (effects (font (size 3 3)) (justify left bottom))
   )
