File: hardware/atf1502as-tqfp44-board/neogeo-diag-mvs-cha-atf1502as-tqfp44.kicad_pcb (KiCad board)
At the start: 2 copper layers, 173.9 x 134 mm, 20 parts, among them J1 neogeo-mvs-cha-a-side-edge, J2 neogeo-mvs-cha-a-side-edge, J3 neogeo-mvs-cha-b-side-edge, J4 neogeo-mvs-cha-b-side-edge, J5 Conn_01x06_Pin, U2 27C010 / 27C1001, U3 27C010 / 27C1001, U4 74HC574, U5 74HC574, U6 ATF1502AS-xAx44

Commit message: Some minor tweaks to schematics and pcbs
Parts:
- J5: value Conn_01x06_Pin -> JTAG
Other:
- board text added: "ATF150xAS"
- board text removed: "ATF1502AS"
