File: hardware/atf1502as-tqfp44-board/neogeo-diag-mvs-cha-atf1502as-tqfp44.kicad_sch (KiCad schematic)
At the start: 18 parts, among them J1 neogeo-mvs-cha-a-side-edge, J2 neogeo-mvs-cha-a-side-edge, J3 neogeo-mvs-cha-b-side-edge, J4 neogeo-mvs-cha-b-side-edge, J5 Conn_01x06_Pin, U2 27C010 / 27C1001, U3 27C010 / 27C1001, U4 74HC574, U5 74HC574, U6 ATF1502AS-xAx44

Commit message: Some minor tweaks to schematics and pcbs
Parts:
- J5: value Conn_01x06_Pin -> JTAG
Other:
- note added: "M1 ROM + Address Logic"
- note removed: "M1 ROM + CPLD (TQFP)"
Changed lines of the file:
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@@
     (effects (font (size 3 3)) (justify left bottom))
   )
-  (text "M1 ROM + CPLD (TQFP)" (at 290.195 149.225 0)
+  (text "M1 ROM + Address Logic" (at 278.765 149.225 0)
     (effects (font (size 3 3)) (justify left bottom))
   )
@@
   )
   (symbol (lib_id "Connector:Conn_01x06_Pin") (at 240.03 205.105 0) (unit 1)
-    (in_bom yes) (on_board yes) (dnp no) (fields_autoplaced)
-    (property "Reference" "J5" (at 240.665 194.945 0)
+    (in_bom yes) (on_board yes) (dnp no)
+    (property "Reference" "J5" (at 245.11 194.31 0)
       (effects (font (size 1.27 1.27)))
     )
-    (property "Value" "Conn_01x06_Pin" (at 240.665 197.485 0)
+    (property "Value" "JTAG" (at 245.11 196.85 0)
       (effects (font (size 1.27 1.27)))
     )
